Commit message: Modified for PhantomX Pincher at PUC-Rio

File: phantomx_arm_description/urdf/phantomx_arm.urdf.xacro (robot description, xacro)
@@ -20,7 +20,5 @@
     <!-- Phantomx arm macro -->
     <phantomx_arm parent="base_link" color="Gray" gripper_color="Gray"   pincher_gripper="true">
-      <!-- Place the "floating" arm at the location it should be if mounted on a turtlebot,
-           as pick and place and other demos assume this location -->
-      <origin xyz="0.1 0.03 0.435"/>
+      <origin xyz="0.0 0.0 0.1"/>
     </phantomx_arm>
 </robot>
