Commit message: Moving to ROS2

File: phantomx_arm_description/urdf/arm_hardware.xacro (robot description, xacro)
@@ -13,5 +13,5 @@
   <xacro:macro name="arm_mount" params="parent name color *origin">
     <joint name="${name}_joint" type="fixed">
-      <insert_block name="origin"/>
+      <xacro:insert_block name="origin"/>
       <parent link="${parent}"/>
       <child link="${name}_link"/>
@@ -47,5 +47,5 @@
   <xacro:macro name="finger_fixed" params="parent name color *origin">
     <joint name="${name}_joint" type="fixed">
-      <insert_block name="origin"/>
+      <xacro:insert_block name="origin"/>
       <parent link="${parent}"/>
       <child link="${name}_link"/>
@@ -81,5 +81,5 @@
   <xacro:macro name="dynamixel_AX12_fixed" params="parent name *origin">
     <joint name="${name}_joint" type="fixed">
-      <insert_block name="origin"/>
+      <xacro:insert_block name="origin"/>
       <parent link="${parent}"/>
       <child link="${name}_link"/>
@@ -115,5 +115,5 @@
   <xacro:macro name="bioloid_F10_fixed" params="parent name color *origin">
     <joint name="${name}_joint" type="fixed">
-      <insert_block name="origin"/>
+      <xacro:insert_block name="origin"/>
       <parent link="${parent}"/>
       <child link="${name}_link"/>
@@ -149,5 +149,5 @@
   <xacro:macro name="bioloid_F3_fixed" params="parent name color *origin">
     <joint name="${name}_joint" type="fixed">
-      <insert_block name="origin"/>
+      <xacro:insert_block name="origin"/>
       <parent link="${parent}"/>
       <child link="${name}_link"/>
@@ -183,5 +183,5 @@
   <xacro:macro name="bioloid_F3_revolute" params="parent name color llimit ulimit vlimit *origin">
     <joint name="${name}_joint" type="revolute">
-      <insert_block name="origin"/>
+      <xacro:insert_block name="origin"/>
       <axis xyz="0 0 -1"/>
       <limit effort="30" velocity="${vlimit}" lower="${llimit}" upper="${ulimit}"/>
@@ -220,5 +220,5 @@
   <xacro:macro name="bioloid_F2_revolute" params="parent name color llimit ulimit vlimit *origin">
     <joint name="${name}_joint" type="revolute">
-      <insert_block name="origin"/>
+      <xacro:insert_block name="origin"/>
       <axis xyz="0 1 0"/>
       <limit effort="30" velocity="${vlimit}" lower="${llimit}" upper="${ulimit}"/>
@@ -257,5 +257,5 @@
   <xacro:macro name="bioloid_F4_revolute" params="parent name color llimit ulimit vlimit *origin">
     <joint name="${name}_joint" type="revolute">
-      <insert_block name="origin"/>
+      <xacro:insert_block name="origin"/>
       <axis xyz="0 1 0"/>
       <limit effort="30" velocity="${vlimit}" lower="${llimit}" upper="${ulimit}"/>
@@ -294,5 +294,5 @@
   <xacro:macro name="gripper_finger_base" params="parent name color *origin">
     <joint name="${name}_joint" type="fixed">
-      <insert_block name="origin"/>
+      <xacro:insert_block name="origin"/>
       <parent link="${parent}"/>
       <child link="${name}_link"/>
@@ -336,5 +336,5 @@
       </inertial>
       <visual>
-        <insert_block name="origin"/>
+        <xacro:insert_block name="origin"/>
         <geometry>
           <mesh filename="package://phantomx_arm_description/meshes/pincher_finger.stl" scale=".01 .01 .01"/>
@@ -343,5 +343,5 @@
       </visual>
       <collision>
-        <insert_block name="origin"/>
+        <xacro:insert_block name="origin"/>
         <geometry>
           <box size="0.036 0.028 0.004"/>

File: phantomx_arm_description/urdf/phantomx_arm.urdf.xacro (robot description, xacro)
@@ -19,6 +19,6 @@
     <link name="base_link"/>
     <!-- Phantomx arm macro -->
-    <phantomx_arm parent="base_link" color="Gray" gripper_color="Gray"   pincher_gripper="true">
+    <xacro:phantomx_arm parent="base_link" color="Gray" gripper_color="Gray"   pincher_gripper="true">
       <origin xyz="0.0 0.0 0.1"/>
-    </phantomx_arm>
+    </xacro:phantomx_arm>
 </robot>

File: phantomx_arm_description/urdf/phantomx_arm.xacro (robot description, xacro)
@@ -18,5 +18,5 @@
     <link name="arm_base_link"/>
     <joint name="arm_base_joint" type="fixed">
-      <insert_block name="origin"/>
+      <xacro:insert_block name="origin"/>
       <parent link="${parent}"/>
       <child link="arm_base_link"/>
@@ -25,68 +25,76 @@
          this makes us 5DOF and saves you $44.90
          that's a lot of coin! -->
+    <link name="gripper_fake_link"/>
+    <joint name="gripper_fake_link_joint" type="revolute">
+      <origin xyz="0 0 0.112" rpy="0 -1.57 0"/>
+      <parent link="arm_wrist_flex_link"/>
+      <child link="gripper_fake_link"/>
+      <limit effort="30" velocity="1.57" lower="-3.14" upper="3.14"/>
+      <axis xyz="1 0 0"/>
+    </joint>
     <link name="gripper_link"/>
     <joint name="gripper_link_joint" type="revolute">
-      <origin xyz="0 0 0.112" rpy="0 -1.57 0"/>
-      <parent link="arm_wrist_flex_link"/>
+      <origin xyz="0 0 0" rpy="0 0 0"/>
+      <parent link="gripper_fake_link"/>
       <child link="gripper_link"/>
-      <limit effort="30" velocity="1" lower="-3.14" upper="3.14"/>
-      <axis xyz="1 0 0"/>
+      <limit effort="30" velocity="1.57" lower="-3.14" upper="3.14"/>
+      <axis xyz="0 0 1"/>
     </joint>
     <!-- shoulder pan joint -->
-    <dynamixel_AX12_fixed parent="arm_base_link" name="arm_shoulder_pan_servo">
+    <xacro:dynamixel_AX12_fixed parent="arm_base_link" name="arm_shoulder_pan_servo">
       <origin xyz="0 0 0" rpy="${M_PI/2} 0 ${M_PI/2}"/>
-    </dynamixel_AX12_fixed>
-    <bioloid_F3_revolute parent="arm_shoulder_pan_servo_link" name="arm_shoulder_pan" color="${color}"
+    </xacro:dynamixel_AX12_fixed>
+    <xacro:bioloid_F3_revolute parent="arm_shoulder_pan_servo_link" name="arm_shoulder_pan" color="${color}"
                          vlimit="${joints_vlimit}" llimit="${pan_llimit}" ulimit="${pan_ulimit}">
       <origin xyz="0 ${AX12_WIDTH/2} 0" rpy="${-M_PI/2} ${M_PI/2} ${M_PI}"/>
-    </bioloid_F3_revolute>
+    </xacro:bioloid_F3_revolute>
     <!-- shoulder lift joint -->
-    <dynamixel_AX12_fixed parent="arm_shoulder_pan_link" name="arm_shoulder_lift_servo">
+    <xacro:dynamixel_AX12_fixed parent="arm_shoulder_pan_link" name="arm_shoulder_lift_servo">
       <origin xyz="0 0 ${-AX12_HEIGHT-F10_HEIGHT+0.001}" rpy="0 ${M_PI} 0"/>
-    </dynamixel_AX12_fixed>
-    <bioloid_F4_revolute parent="arm_shoulder_lift_servo_link" name="arm_shoulder_lift" color="${color}"
+    </xacro:dynamixel_AX12_fixed>
+    <xacro:bioloid_F4_revolute parent="arm_shoulder_lift_servo_link" name="arm_shoulder_lift" color="${color}"
                          vlimit="${joints_vlimit}" llimit="${shoulder_llimit}" ulimit="${shoulder_ulimit}">
       <origin xyz="0 0 0" rpy="0 0 0"/>
-    </bioloid_F4_revolute>
-    <bioloid_F10_fixed parent="arm_shoulder_lift_link" name="arm_shoulder_F10_0" color="${color}">
+    </xacro:bioloid_F4_revolute>
+    <xacro:bioloid_F10_fixed parent="arm_shoulder_lift_link" name="arm_shoulder_F10_0" color="${color}">
       <origin xyz="0 0 ${F4_HEIGHT+F10_HEIGHT/2}" rpy="0 0 0"/>
-    </bioloid_F10_fixed>
-    <bioloid_F10_fixed parent="arm_shoulder_F10_0_link" name="arm_shoulder_F10_1" color="${color}">
+    </xacro:bioloid_F10_fixed>
+    <xacro:bioloid_F10_fixed parent="arm_shoulder_F10_0_link" name="arm_shoulder_F10_1" color="${color}">
       <origin xyz="0 0 ${F10_HEIGHT}" rpy="0 0 0"/>
-    </bioloid_F10_fixed>
-    <bioloid_F10_fixed parent="arm_shoulder_F10_1_link" name="arm_shoulder_F10_2" color="${color}">
+    </xacro:bioloid_F10_fixed>
+    <xacro:bioloid_F10_fixed parent="arm_shoulder_F10_1_link" name="arm_shoulder_F10_2" color="${color}">
       <origin xyz="0 0 ${F10_HEIGHT}" rpy="0 0 0"/>
-    </bioloid_F10_fixed>
-    <bioloid_F3_fixed parent="arm_shoulder_F10_2_link" name="arm_shoulder_F3_0" color="${color}">
+    </xacro:bioloid_F10_fixed>
+    <xacro:bioloid_F3_fixed parent="arm_shoulder_F10_2_link" name="arm_shoulder_F3_0" color="${color}">
       <origin xyz="0 0 ${F10_HEIGHT/2}" rpy="0 ${M_PI} 0"/>
-    </bioloid_F3_fixed>
+    </xacro:bioloid_F3_fixed>
     <!-- elbow joint -->
-    <dynamixel_AX12_fixed parent="arm_shoulder_F3_0_link" name="arm_elbow_flex_servo">
+    <xacro:dynamixel_AX12_fixed parent="arm_shoulder_F3_0_link" name="arm_elbow_flex_servo">
       <origin xyz="0 0 ${-AX12_HEIGHT-F10_HEIGHT+0.001}" rpy="0 ${M_PI} 0"/>
-    </dynamixel_AX12_fixed>
-    <bioloid_F4_revolute parent="arm_elbow_flex_servo_link" name="arm_elbow_flex" color="${color}"
+    </xacro:dynamixel_AX12_fixed>
+    <xacro:bioloid_F4_revolute parent="arm_elbow_flex_servo_link" name="arm_elbow_flex" color="${color}"
                          vlimit="${joints_vlimit}" llimit="${elbow_llimit}" ulimit="${elbow_ulimit}">
       <origin xyz="0 0 0" rpy="0 0 0"/>
-    </bioloid_F4_revolute>
-    <bioloid_F10_fixed parent="arm_elbow_flex_link" name="arm_elbow_F10_0" color="${color}">
+    </xacro:bioloid_F4_revolute>
+    <xacro:bioloid_F10_fixed parent="arm_elbow_flex_link" name="arm_elbow_F10_0" color="${color}">
       <origin xyz="0 0 ${F4_HEIGHT+F10_HEIGHT/2}" rpy="0 0 0"/>
-    </bioloid_F10_fixed>
-    <bioloid_F10_fixed parent="arm_elbow_F10_0_link" name="arm_elbow_F10_1" color="${color}">
+    </xacro:bioloid_F10_fixed>
+    <xacro:bioloid_F10_fixed parent="arm_elbow_F10_0_link" name="arm_elbow_F10_1" color="${color}">
       <origin xyz="0 0 ${F10_HEIGHT}" rpy="0 0 0"/>
-    </bioloid_F10_fixed>
-    <bioloid_F10_fixed parent="arm_elbow_F10_1_link" name="arm_elbow_F10_2" color="${color}">
+    </xacro:bioloid_F10_fixed>
+    <xacro:bioloid_F10_fixed parent="arm_elbow_F10_1_link" name="arm_elbow_F10_2" color="${color}">
       <origin xyz="0 0 ${F10_HEIGHT}" rpy="0 0 0"/>
-    </bioloid_F10_fixed>
-    <bioloid_F3_fixed parent="arm_elbow_F10_2_link" name="arm_elbow_F3_0" color="${color}">
+    </xacro:bioloid_F10_fixed>
+    <xacro:bioloid_F3_fixed parent="arm_elbow_F10_2_link" name="arm_elbow_F3_0" color="${color}">
       <origin xyz="0 0 ${F10_HEIGHT/2}" rpy="0 ${M_PI} 0"/>
-    </bioloid_F3_fixed>
+    </xacro:bioloid_F3_fixed>
     <!-- wrist joint -->
-    <dynamixel_AX12_fixed parent="arm_elbow_F3_0_link" name="arm_wrist_flex_servo">
+    <xacro:dynamixel_AX12_fixed parent="arm_elbow_F3_0_link" name="arm_wrist_flex_servo">
       <origin xyz="0 0 ${-AX12_HEIGHT-F10_HEIGHT+0.001}" rpy="0 ${M_PI} 0"/>
-    </dynamixel_AX12_fixed>
-    <bioloid_F2_revolute parent="arm_wrist_flex_servo_link" name="arm_wrist_flex" color="${color}"
+    </xacro:dynamixel_AX12_fixed>
+    <xacro:bioloid_F2_revolute parent="arm_wrist_flex_servo_link" name="arm_wrist_flex" color="${color}"
                          vlimit="${joints_vlimit}" llimit="${wrist_llimit}" ulimit="${wrist_ulimit}">
       <origin xyz="0 0 0" rpy="0 0 0"/>
-    </bioloid_F2_revolute>
+    </xacro:bioloid_F2_revolute>
   <!-- gripper - Pincher Gripper -->
   <xacro:include filename="$(find phantomx_arm_description)/urdf/phantomx_gripper.xacro"/>

File: phantomx_arm_description/urdf/phantomx_gripper.xacro (robot description, xacro)
@@ -2,14 +2,14 @@
 <!-- PhantomX Pincher Arm gripper URDF-->
 <robot xmlns:xacro="http://ros.org/wiki/xacro">
-    <bioloid_F3_fixed parent="arm_wrist_flex_link" name="arm_wrist_F3_0" color="${color}">
+    <xacro:bioloid_F3_fixed parent="arm_wrist_flex_link" name="arm_wrist_F3_0" color="${color}">
       <origin xyz="0 0 ${F2_HEIGHT}" rpy="0 ${M_PI} ${-M_PI}"/>
-    </bioloid_F3_fixed>
+    </xacro:bioloid_F3_fixed>
     <!-- gripper joint -->
-    <dynamixel_AX12_fixed parent="arm_wrist_F3_0_link" name="gripper_servo" >
+    <xacro:dynamixel_AX12_fixed parent="arm_wrist_F3_0_link" name="gripper_servo" >
       <origin xyz="0 0 ${-AX12_WIDTH/2}" rpy="${M_PI/2} ${M_PI} ${M_PI/2}"/>
-    </dynamixel_AX12_fixed>
-     <gripper_finger_base parent="gripper_servo_link" name="gripper_finger_base" color="${color}">
+    </xacro:dynamixel_AX12_fixed>
+     <xacro:gripper_finger_base parent="gripper_servo_link" name="gripper_finger_base" color="${color}">
       <origin xyz="0.01  ${AX12_WIDTH} 0" rpy="${M_PI/2} ${-M_PI} ${M_PI/2}"/>
-    </gripper_finger_base>
+    </xacro:gripper_finger_base>
      <!-- Finger 1 -->
     <joint name="gripper_joint" type="prismatic">
@@ -20,7 +20,7 @@
       <child link="gripper_active_link"/>
     </joint>
-    <pincher_gripper name="gripper_active" color="${color}" >
+    <xacro:pincher_gripper name="gripper_active" color="${color}" >
       <origin xyz="-0.02 0.023 0" rpy="${-M_PI/2} 0 0"/>
-    </pincher_gripper>
+    </xacro:pincher_gripper>
     <!-- Finger 2 -->
     <!-- Note: currently static but should be a Mimic of Finger 1 -->
@@ -29,7 +29,7 @@
       <child link="gripper_active2_link"/>
     </joint>
-    <pincher_gripper name="gripper_active2" color="${color}" >
+    <xacro:pincher_gripper name="gripper_active2" color="${color}" >
       <origin xyz="-0.02 0.023 0" rpy="${-M_PI/2} ${M_PI} 0"/>
-    </pincher_gripper>
+    </xacro:pincher_gripper>
     <!-- Using Mimic -->
     <!-- gripper 2 joint -->
