Commit message: Better error handling

File: phantomx_arm_description/urdf/phantomx_gripper.xacro (robot description, xacro)
@@ -16,5 +16,5 @@
       <origin xyz="0 0 0" rpy="0 0 0"/>
       <axis xyz="1 0 0"/>
-      <limit effort="30" velocity="0.5" lower="0.002" upper="0.031"/>
+      <limit effort="30" velocity="0.5" lower="-2.0" upper="2.0"/>
       <parent link="gripper_servo_link"/>
       <child link="gripper_active_link"/>

Commit message: Set gripper position in cm (0 = open, -0.02 = closed)

File: phantomx_arm_description/urdf/phantomx_gripper.xacro (robot description, xacro)
@@ -14,7 +14,7 @@
      <!-- Finger 1 -->
     <joint name="gripper_joint" type="prismatic">
-      <origin xyz="0 0 0" rpy="0 0 0"/>
+      <origin xyz="0.03 0 0" rpy="0 0 0"/>
       <axis xyz="1 0 0"/>
-      <limit effort="30" velocity="0.5" lower="-2.0" upper="2.0"/>
+      <limit effort="30" velocity="0.005" lower="-0.021" upper="0.001"/>
       <parent link="gripper_servo_link"/>
       <child link="gripper_active_link"/>
